Commit message: working sensors

File: src/my_robot/urdf/my_robot.xacro (robot description, xacro)
@@ -1,19 +1,5 @@
 <?xml version='1.0'?>
 <robot name="my_robot" xmlns:xacro="http://www.ros.org/wiki/xacro">
-  <material name="blue">
-    <color rgba="0.0 0.0 0.8 1.0"/>
-  </material>
-  <material name="green">
-    <color rgba="0.0 0.8 0.0 1.0"/>
-  </material>
-  <material name="gray">
-    <color rgba="0.7 0.7 0.7 1.0"/>
-  </material>
-  <material name="darkgray">
-    <color rgba="0.3 0.3 0.3 1.0"/>
-  </material>
-  <material name="red">
-    <color rgba="0.8 0.0 0.0 1.0"/>
-  </material>
+  <xacro:include filename="$(find my_robot)/urdf/my_robot.gazebo" />
   <link name="robot_footprint"></link>
   <joint name="robot_footprint_joint" type="fixed">
@@ -71,4 +57,7 @@
     </visual>
   </link>
+  <gazebo reference="chassis">
+    <material>Gazebo/Blue</material>
+  </gazebo>
   <link name='left_wheel'>
     <inertial>
@@ -92,7 +81,9 @@
         <cylinder radius=".1" length=".05"/>
       </geometry>
-      <material name="green"/>
     </visual>
   </link>
+  <gazebo reference="left_wheel">
+    <material>Gazebo/Red</material>
+  </gazebo>
   <link name='right_wheel'>
     <inertial>
@@ -116,7 +107,9 @@
         <cylinder radius=".1" length=".05"/>
       </geometry>
-      <material name="green"/>
     </visual>
   </link>
+  <gazebo reference="right_wheel">
+    <material>Gazebo/Red</material>
+  </gazebo>
   <joint type="continuous" name="left_wheel_hinge">
     <origin xyz="0 0.15 0" rpy="0 0 0"/>

Commit message: adding the RGB-D camera

File: src/my_robot/urdf/my_robot.xacro (robot description, xacro)
@@ -190,3 +190,10 @@
     <dynamics damping="1.0" friction="1.0"/>
   </joint>
+  <joint name="camera_optical_joint" type="fixed">
+    <origin xyz="0 0 0" rpy="-1.5707 0 -1.5707"/>
+    <parent link="camera"/>
+    <child link="camera_link_optical"/>
+  </joint>
+  <link name="camera_link_optical">
+  </link>
 </robot>
